Commit message: change description package to latest state (ros2 control definitions included)

File: src/sew_agv_description/urdf/sew_agv_macro.urdf.xacro (robot description, xacro)
@@ -14,6 +14,5 @@
     ros2_control_with_gazebo:=false
     use_fake_hardware:=false
-    robot_ip
-    robot_ssid"
+    robot_ip"
   >
 <!--#######################################################################################################################################-->
@@ -22,19 +21,26 @@
     <xacro:if value="${generate_ros2_control_tag}">
         <!-- ros2 control include -->
-        <xacro:include filename="$(find sew_agv_description)/urdf/sew_agv.ros2_control.urdf.xacro" />
+        <xacro:include filename="$(find sew_agv_description)/urdf/sew_agv_ros2_control.urdf.xacro" />
         <!-- ros2 control instance -->
         <xacro:sew_agv_ros2_control
           ros2_control_with_gazebo="${ros2_control_with_gazebo}"
+          use_fake_hardware="${use_fake_hardware}"
           tf_prefix="${tf_prefix}"
-          robot_ip="${robot_ip}"
-          robot_ssid="${robot_ssid}"
+          agv_ip="${robot_ip}"
         />
     </xacro:if>
 <!--#######################################################################################################################################-->
-<!--load gazebo hardware plugin for ros2_control or standard gazebo diff_drive plugin-->
+<!--load standard gazebo diff_drive plugin-->
 <!--#######################################################################################################################################-->
     <xacro:if value="${standalone_gazebo}">
         <xacro:include filename="$(find sew_agv_description)/urdf/sew_agv_gazebo_macro.urdf.xacro" />
-        <xacro:sew_agv_gazebo/>
+        <xacro:sew_agv_gazebo tf_prefix="${tf_prefix}"/>
+    </xacro:if>
+<!--#######################################################################################################################################-->
+<!--load gazebo hardware plugin for ros2_control diff_drive plugin-->
+<!--#######################################################################################################################################-->
+    <xacro:if value="${ros2_control_with_gazebo}">
+        <xacro:include filename="$(find sew_agv_description)/urdf/sew_agv_ros2_control_gazebo_macro.urdf.xacro" />
+        <xacro:sew_ros2_control_gazebo tf_prefix="${tf_prefix}"/>
     </xacro:if>
 <!--#######################################################################################################################################-->

File: src/sew_agv_description/urdf/sew_agv_model.urdf.xacro (robot description, xacro)
@@ -9,10 +9,9 @@
     <!-- set ros2 parameters, which will passsed to the macros, can be defined in the launch file-->
 <!--#######################################################################################################################################-->
-   <!-- set parameters defined in diy_robotarm_macro.xacro -->
+   <!-- set parameters defined in sew_agv_macro.xacro -->
     <xacro:arg name="tf_prefix" default=""/>
     <!-- ros2_control related parameters -->
     <xacro:arg name="robot_ip" default="NaN" />
-    <xacro:arg name="robot_ssid" default="NaN" />
-    <xacro:arg name="generate_ros2_control_tag" default="false" />
+    <xacro:arg name="generate_ros2_control_tag" default="true" />               <!--change default value ??? seems to be not passed to here-->
     <!-- simulation related parameters -->
     <xacro:arg name="use_fake_hardware" default="false" />
@@ -27,5 +26,4 @@
         use_fake_hardware="$(arg use_fake_hardware)"
         robot_ip="$(arg robot_ip)"
-        robot_ssid="$(arg robot_ssid)"
         generate_ros2_control_tag="$(arg generate_ros2_control_tag)"
         standalone_gazebo="$(arg standalone_gazebo)"

File: src/sew_agv_description/urdf/sew_agv_ros2_control_gazebo_macro.urdf.xacro (robot description, xacro)
@@ -1,30 +1,16 @@
 <?xml version="1.0"?>
 <robot xmlns:xacro="http://www.ros.org/wiki/xacro">
-    <xacro:macro name="sew_agv_gazebo" params="tf_prefix">
+    <xacro:macro name="sew_ros2_control_gazebo" params="tf_prefix">
     <!--#######################################################################################################################################-->
-    <!--set up the diff_drive plugin controller from gazebo, NOT ros2_control -> maybe change when ros2_control available -->
+    <!--set up the ros2 control plugin for the sew diff drive controller-->
     <!--#######################################################################################################################################-->
-        <gazebo>
-            <plugin name="diff_drive" filename="libgazebo_ros_diff_drive.so">
-                <update_rate>30</update_rate>
-                <!--set wheels-->
-                <left_joint>sew_wheel_left_joint</left_joint>
-                <right_joint>sew_wheel_right_joint</right_joint>
-                <wheel_separation>0.525</wheel_separation>
-                <wheel_diameter>0.2</wheel_diameter>
-                <!-- joint limits/ overrides urdf definitions ! -->
-                <max_wheel_torque>20</max_wheel_torque>
-                <max_wheel_acceleration>1.0</max_wheel_acceleration>
-                <!-- Output messages of the plugin gazebo -> ros2-->
-                <odometry_frame>odom</odometry_frame>
-                <robot_base_frame>sew_base_footprint</robot_base_frame>
-                <publish_odom>true</publish_odom>
-                <publish_odom_tf>true</publish_odom_tf>
-                <publish_wheel_tf>true</publish_wheel_tf>
-                <!--command topic ros2 -> gazebo-->
-                <command_topic>cmd_vel_out</command_topic>      <!--whyever this has no effect on gazebo -> remap topics in launch file-->
-            </plugin>
-        </gazebo>
-        <!--later add ros2 control plugin : https://www.youtube.com/watch?v=4QKsDf1c4hc&list=PLunhqkrRNRhYAffV8JDiFOatQXuU-NnxT&index=12-->
+    <gazebo>
+        <plugin filename="libgazebo_ros2_control.so" name="gazebo_ros2_control">
+          <robot_param>robot_description</robot_param>
+          <robot_param_node>robot_state_publisher</robot_param_node>
+          <parameters>$(find sew_agv_drivers)/config/agv_controller.yaml</parameters>
+          <controller_manager_name>controller_manager</controller_manager_name>
+        </plugin>
+    </gazebo>
     <!--#######################################################################################################################################-->
     <!--define gazebo tags for materials, because urdf materialc can not be used in gazebo -->
