Commit message: load new descriprion package and change names with tf_prefix

File: src/sew_agv_description/urdf/sew_agv_gazebo_macro.urdf.xacro (robot description, xacro)
@@ -9,6 +9,6 @@
                 <update_rate>30</update_rate>
                 <!--set wheels-->
-                <left_joint>wheel_left_joint</left_joint>
-                <right_joint>wheel_right_joint</right_joint>
+                <left_joint>sew_wheel_left_joint</left_joint>
+                <right_joint>sew_wheel_right_joint</right_joint>
                 <wheel_separation>0.525</wheel_separation>
                 <wheel_diameter>0.2</wheel_diameter>
@@ -18,5 +18,5 @@
                 <!-- Output messages of the plugin gazebo -> ros2-->
                 <odometry_frame>odom</odometry_frame>
-                <robot_base_frame>base_footprint</robot_base_frame>
+                <robot_base_frame>sew_base_footprint</robot_base_frame>
                 <publish_odom>true</publish_odom>
                 <publish_odom_tf>true</publish_odom_tf>
@@ -30,17 +30,17 @@
     <!--define gazebo tags for materials, because urdf materialc can not be used in gazebo -->
     <!--#######################################################################################################################################-->
-        <gazebo reference="caster_wheel_link">
+        <gazebo reference="sew_caster_wheel_link">
             <material> Gazebo/Black</material>
         </gazebo>
-        <gazebo reference="right_wheel_link">
+        <gazebo reference="sew_right_wheel_link">
             <material> Gazebo/Black</material>
         </gazebo>
-        <gazebo reference="left_wheel_link">
+        <gazebo reference="sew_left_wheel_link">
             <material> Gazebo/Black</material>
         </gazebo>
-        <gazebo reference="body_link">
+        <gazebo reference="sew_body_link">
             <material> Gazebo/Grey</material>
         </gazebo>
-        <gazebo reference="lidar_link">
+        <gazebo reference="sew_lidar_link">
             <material> Gazebo/Yellow</material>
         </gazebo>
@@ -48,5 +48,5 @@
     <!--set friction of the caster wheel to nearly 0 (for simplicity reasons) -->
     <!--#######################################################################################################################################-->
-        <gazebo reference="caster_wheel_link">
+        <gazebo reference="sew_caster_wheel_link">
             <mu1 value="0.001"/>
             <mu2 value="0.001"/>
@@ -55,5 +55,5 @@
     <!--include lidar sensor simulation on lidar link -->
     <!--#######################################################################################################################################-->
-        <gazebo reference="lidar_link">
+        <gazebo reference="sew_lidar_link">
             <sensor type="ray" name="lidar_1">
                 <pose> 0 0 0 0 0 0 </pose>      <!--define offset to lidar_link frame-->

File: src/sew_agv_description/urdf/sew_agv_macro.urdf.xacro (robot description, xacro)
@@ -25,5 +25,5 @@
         <!-- ros2 control instance -->
         <xacro:sew_agv_ros2_control
-          use_fake_hardware="${use_fake_hardware}"
+          ros2_control_with_gazebo="${ros2_control_with_gazebo}"
           tf_prefix="${tf_prefix}"
           robot_ip="${robot_ip}"
@@ -34,9 +34,4 @@
 <!--load gazebo hardware plugin for ros2_control or standard gazebo diff_drive plugin-->
 <!--#######################################################################################################################################-->
-    <xacro:if value="${ros2_control_with_gazebo}">
-        <hardware>
-            <plugin>gz_ros2_control/GazeboSimSystem</plugin>
-        </hardware>
-    </xacro:if>
     <xacro:if value="${standalone_gazebo}">
         <xacro:include filename="$(find sew_agv_description)/urdf/sew_agv_gazebo_macro.urdf.xacro" />
@@ -48,17 +43,17 @@
     <xacro:materials tf_prefix="${tf_prefix}"/>
     <!--define non physical footprint joint (used in nav2 to determine robot center on the ground)-->
-    <link name="base_footprint"/>
+    <link name="${tf_prefix}base_footprint"/>
     <!--base/ main body fixed relative to the footprint , inertial definitions required due to the use in gazebo-->
-    <joint name="base_footprint_joint" type="fixed">
+    <joint name="${tf_prefix}base_footprint_joint" type="fixed">
         <origin rpy="0 0 0" xyz="0 0 0.58"/>
         <axis xyz="0 0 0"/>
-        <parent link="base_footprint"/>
-        <child link="base_link"/>
+        <parent link="${tf_prefix}base_footprint"/>
+        <child link="${tf_prefix}base_link"/>
     </joint>
-    <link name="base_link">
+    <link name="${tf_prefix}base_link">
         <inertial>
             <mass value="250"/> <!--in kg-->
             <origin rpy="0 0 0" xyz="0 0 0"/>
-            <inertia ixx="3.82" ixy="0.0" ixz="0.48" iyy="4.11" iyz="0.0" izz="3.29"/> <!--not realistic!-->
+            <inertia ixx="1.0" ixy="0.0" ixz="0.0" iyy="1.0" iyz="0.0" izz="1.0"/> <!--not realistic!-->
         </inertial>
         <visual>
@@ -78,14 +73,14 @@
     </link>
     <!--front wheel / axis should match the rotation axis of the wheel, for simplicity reasons set this to fixed and disable friction in gazebo-->
-    <joint name="caster_wheel_joint" type="fixed">
+    <joint name="${tf_prefix}caster_wheel_joint" type="fixed">
         <origin rpy="1.57079 0 0" xyz="0.290 0 -0.56"/>
         <axis xyz="0 0 0"/>
-        <parent link="base_link"/>
-        <child link="caster_wheel_link"/>
+        <parent link="${tf_prefix}base_link"/>
+        <child link="${tf_prefix}caster_wheel_link"/>
     </joint>
-    <link name="caster_wheel_link" type="wheel">
+    <link name="${tf_prefix}caster_wheel_link" type="wheel">
         <inertial>
             <mass value="2"/>
-            <inertia ixx="0.0" ixy="0.0" ixz="0.0" iyy="1.0" iyz="0.0" izz="1.0"/> <!--not realistic!-->
+            <inertia ixx="1.0" ixy="0.0" ixz="0.0" iyy="1.0" iyz="0.0" izz="1.0"/> <!--not realistic!-->
         </inertial>
         <visual>
@@ -105,17 +100,16 @@
     </link>
     <!--right back wheel / axis shold match the rotation axis of the wheel-->
-    <joint name="wheel_right_joint" type="continuous">
+    <joint name="${tf_prefix}wheel_right_joint" type="continuous">
         <origin rpy="0 0 -1.57079" xyz="-0.225 -0.2625 -0.48"/>
         <limit effort="100.0" velocity="3.5"/>
         <axis xyz="-1 0 0"/>
-        <parent link="base_link"/>
-        <child link="wheel_right_link"/>
-        <joint_properties damping="1" friction="1"/>
+        <parent link="${tf_prefix}base_link"/>
+        <child link="${tf_prefix}wheel_right_link"/>
     </joint>
-    <link name="wheel_right_link" type="wheel">
+    <link name="${tf_prefix}wheel_right_link" type="wheel">
         <inertial>
             <origin rpy="0 0 0" xyz="0 0 0"/>
             <mass value="2"/>
-            <inertia ixx="0.0" ixy="0.0" ixz="0.0" iyy="1.0" iyz="0.0" izz="1.0"/> <!--not realistic!-->
+            <inertia ixx="1.0" ixy="0.0" ixz="0.0" iyy="1.0" iyz="0.0" izz="1.0"/> <!--not realistic!-->
         </inertial>
         <visual>
@@ -135,13 +129,12 @@
     </link>
     <!--left back wheel / axis shold match the rotation axis of the wheel-->
-    <joint name="wheel_left_joint" type="continuous">
+    <joint name="${tf_prefix}wheel_left_joint" type="continuous">
         <origin rpy="0 0 1.57079" xyz="-0.225 0.2625 -0.48"/>
         <limit effort="100.0" velocity="3.5"/>
         <axis xyz="1 0 0"/>
-        <parent link="base_link"/>
-        <child link="wheel_left_link"/>
-        <joint_properties damping="5" friction="10"/>
+        <parent link="${tf_prefix}base_link"/>
+        <child link="${tf_prefix}wheel_left_link"/>
     </joint>
-    <link name="wheel_left_link" type="wheel">
+    <link name="${tf_prefix}wheel_left_link" type="wheel">
         <inertial>
             <origin rpy="0 0 0" xyz="0 0 0"/>
@@ -165,11 +158,11 @@
     </link>
     <!--lidar sensor, required due to the use in gazebo-->
-    <joint name="lidar_joint" type="fixed">
+    <joint name="${tf_prefix}lidar_joint" type="fixed">
         <axis xyz="0 0 0"/>
         <origin rpy="0 0 0 " xyz="0.355 0 -0.445"/>
-        <parent link="base_link"/>
-        <child link="lidar_link"/>
+        <parent link="${tf_prefix}base_link"/>
+        <child link="${tf_prefix}lidar_link"/>
     </joint>
-    <link name="lidar_link" type="laser">
+    <link name="${tf_prefix}lidar_link" type="laser">
         <inertial>
             <mass value="1"/>

Commit message: fix sliding in sim by reducing weight

File: src/sew_agv_description/urdf/sew_agv_gazebo_macro.urdf.xacro (robot description, xacro)
@@ -49,6 +49,6 @@
     <!--#######################################################################################################################################-->
         <gazebo reference="${tf_prefix}caster_wheel_link">
-            <mu1 value="0.001"/>
-            <mu2 value="0.001"/>
+            <mu1 value="1000"/>
+            <mu2 value="1000"/>
         </gazebo>
     <!--#######################################################################################################################################-->

File: src/sew_agv_description/urdf/sew_agv_macro.urdf.xacro (robot description, xacro)
@@ -59,6 +59,6 @@
     <link name="${tf_prefix}base_link">
         <inertial>
-            <mass value="250"/> <!--in kg-->
-            <origin rpy="0 0 0" xyz="0 0 0"/>
+            <mass value="50"/> <!--in kg reduced due to simulation instabilities at higher weight-->
+            <origin rpy="0 0 -0.5" xyz="0 0 0"/>
             <inertia ixx="1.0" ixy="0.0" ixz="0.0" iyy="1.0" iyz="0.0" izz="1.0"/> <!--not realistic!-->
         </inertial>
