Commit message: edit srdf

File: src/sew_and_igus_moveit_config/srdf/igus_rebel_6dof.srdf.xacro (robot description, xacro)
@@ -2,7 +2,7 @@
 <robot xmlns:xacro="http://wiki.ros.org/xacro"
        name="igus_rebel_6dof" >
-    <xacro:arg name="prefix" default="" />
+    <xacro:arg name="prefix" default="igus_" />
+    <xacro:arg name="tf_prefix" default="sew_" />
     <group name="rebel_6dof">
-        <link name="world"/>
         <link name="$(arg prefix)base_link"/>
         <link name="$(arg prefix)link_1"/>
@@ -19,5 +19,5 @@
         <joint name="$(arg prefix)joint6"/>
         <joint name="$(arg prefix)joint7"/>
-        <chain base_link="world" tip_link="$(arg prefix)link_8"/>
+        <chain base_link="$(arg prefix)base_link" tip_link="$(arg prefix)link_8"/>
     </group>
     <group_state name="zero" group="rebel_6dof">
@@ -29,5 +29,7 @@
         <joint name="$(arg prefix)joint6" value="0"/>
     </group_state>
-    <virtual_joint name="world_to_base" type="fixed" parent_frame="world" child_link="$(arg prefix)base_link"/>
+    <virtual_joint name="world_to_base" type="fixed" parent_frame="world" child_link="$(arg tf_prefix)base_footprint"/>
+    <!--sew to igus connection is not a collision-->
+    <disable_collisions link1="$(arg tf_prefix)base_link" link2="$(arg prefix)base_link" reason="Adjacent"/>
     <disable_collisions link1="$(arg prefix)base_link" link2="$(arg prefix)link_1" reason="Adjacent"/>
     <disable_collisions link1="$(arg prefix)gripper_base" link2="$(arg prefix)gripper_mount" reason="Adjacent"/>

Commit message: add tool0 to serial chain

File: src/sew_and_igus_moveit_config/srdf/igus_rebel_6dof.srdf.xacro (robot description, xacro)
@@ -12,4 +12,5 @@
         <link name="$(arg prefix)link_7"/>
         <link name="$(arg prefix)link_8"/>
+        <link name="$(arg prefix)tool0"/>
         <joint name="$(arg prefix)joint1"/>
         <joint name="$(arg prefix)joint2"/>
@@ -19,5 +20,5 @@
         <joint name="$(arg prefix)joint6"/>
         <joint name="$(arg prefix)joint7"/>
-        <chain base_link="$(arg prefix)base_link" tip_link="$(arg prefix)link_8"/>
+        <chain base_link="$(arg prefix)base_link" tip_link="$(arg prefix)tool0"/>
     </group>
     <group_state name="zero" group="rebel_6dof">

Commit message: delete joint and link definitions in group

File: src/sew_and_igus_moveit_config/srdf/igus_rebel_6dof.srdf.xacro (robot description, xacro)
@@ -5,19 +5,4 @@
     <xacro:arg name="tf_prefix" default="sew_" />
     <group name="rebel_6dof">
-        <link name="$(arg prefix)base_link"/>
-        <link name="$(arg prefix)link_1"/>
-        <link name="$(arg prefix)link_2"/>
-        <link name="$(arg prefix)link_5"/>
-        <link name="$(arg prefix)link_6"/>
-        <link name="$(arg prefix)link_7"/>
-        <link name="$(arg prefix)link_8"/>
-        <link name="$(arg prefix)tool0"/>
-        <joint name="$(arg prefix)joint1"/>
-        <joint name="$(arg prefix)joint2"/>
-        <joint name="$(arg prefix)joint3"/>
-        <joint name="$(arg prefix)joint4"/>
-        <joint name="$(arg prefix)joint5"/>
-        <joint name="$(arg prefix)joint6"/>
-        <joint name="$(arg prefix)joint7"/>
         <chain base_link="$(arg prefix)base_link" tip_link="$(arg prefix)tool0"/>
     </group>
