Commit message: add collission geommetry to camera link

File: src/sew_and_igus_description/urdf/gazebo_depth_camera_macro.urdf.xacro (robot description, xacro)
@@ -17,4 +17,10 @@
                 <material name="${prefix}yellow"/>
             </visual>
+            <collision>
+                <geometry>
+                    <box size="0.03 0.03 0.03"/>
+                </geometry>
+                <material name="${prefix}red"/>
+            </collision>
         </link>
         <joint name="${prefix}camera_optical_joint" type="fixed">
