Commit message: add schaltschrank and adapter plate to urdf

File: src/sew_and_igus_description/urdf/sew_and_igus_model.urdf.xacro (robot description, xacro)
@@ -26,4 +26,63 @@
     </xacro:sew_agv_macro>
 <!--#######################################################################################################################################-->
+   <!-- add adapter plate and cabinet -->
+<!--#######################################################################################################################################-->
+    <xacro:include filename="$(find sew_and_igus_description)/urdf/materials.urdf.xacro" />
+    <xacro:materials tf_prefix=""/>
+    <joint name="sew_to_adapterplate" type="fixed">
+        <origin rpy="0 0 1.57" xyz="-0.29 0 0"/>
+        <axis xyz="0 0 0"/>
+        <parent link="$(arg tf_prefix)base_link"/>
+        <child link="adapterplate_link"/>
+    </joint>
+    <link name="adapterplate_link">
+        <inertial>
+            <mass value="2"/> <!--in kg reduced due to simulation instabilities at higher weight-->
+            <origin rpy="0 0 0" xyz="0 0 0"/>
+            <inertia ixx="1.0" ixy="0.0" ixz="0.0" iyy="1.0" iyz="0.0" izz="1.0"/> <!--not realistic!-->
+        </inertial>
+        <visual>
+            <origin rpy="0 0 0" xyz="0 0 0"/>
+            <geometry>
+                <mesh filename="file://$(find sew_and_igus_description)/meshes/visual/adapter_plate.stl" scale="0.001 0.001 0.001"/>
+            </geometry>
+            <material name="grey"/>
+        </visual>
+        <collision>
+            <origin rpy=" 0 0 0" xyz="0 0 0"/>
+            <geometry>
+                <mesh filename="file://$(find sew_and_igus_description)/meshes/collision/adapter_plate.stl" scale="0.001 0.001 0.001"/>
+            </geometry>
+            <material name="red"/>
+        </collision>
+    </link>
+    <joint name="adapterplate_to_cabinet" type="fixed">
+        <origin rpy="0 0 0" xyz="-0.095 -0.005 0.023"/>
+        <axis xyz="0 0 0"/>
+        <parent link="adapterplate_link"/>
+        <child link="cabinet_link"/>
+    </joint>
+    <link name="cabinet_link">
+        <inertial>
+            <mass value="3"/> <!--in kg reduced due to simulation instabilities at higher weight-->
+            <origin rpy="0 0 0" xyz="0 0 0"/>
+            <inertia ixx="1.0" ixy="0.0" ixz="0.0" iyy="1.0" iyz="0.0" izz="1.0"/> <!--not realistic!-->
+        </inertial>
+        <visual>
+            <origin rpy="0 0 0" xyz="0 0 0"/>
+            <geometry>
+                <mesh filename="file://$(find sew_and_igus_description)/meshes/visual/schaltschrank.stl" scale="0.001 0.001 0.001"/>
+            </geometry>
+            <material name="grey"/>
+        </visual>
+        <collision>
+            <origin rpy=" 0 0 0" xyz="0 0 0"/>
+            <geometry>
+                <mesh filename="file://$(find sew_and_igus_description)/meshes/collision/schaltschrank.stl" scale="0.001 0.001 0.001"/>
+            </geometry>
+            <material name="red"/>
+        </collision>
+    </link>
+<!--#######################################################################################################################################-->
    <!-- import igus-macro, define parameters needed inside the macro and load the macro -->
 <!--#######################################################################################################################################-->
@@ -48,8 +107,8 @@
    <!-- joint which connects the sew agv and the igus arm -->
 <!--#######################################################################################################################################-->
-  <joint name="sew_to_$(arg prefix)base" type="fixed">
-    <parent link="$(arg tf_prefix)base_link" />
+  <joint name="adapterplate_to_$(arg prefix)base" type="fixed">
+    <parent link="adapterplate_link" />
     <child link = "$(arg prefix)base_link" />
-    <origin xyz="0 0 0" rpy="0 0 0" />
+    <origin xyz="0.19 -0.015 0.023" rpy="0 0 -1.57" />
   </joint>
 </robot>

Commit message: rotate robot by 180 deg.

File: src/sew_and_igus_description/urdf/sew_and_igus_model.urdf.xacro (robot description, xacro)
@@ -110,5 +110,5 @@
     <parent link="adapterplate_link" />
     <child link = "$(arg prefix)base_link" />
-    <origin xyz="0.19 -0.015 0.023" rpy="0 0 -1.57" />
+    <origin xyz="0.19 -0.015 0.023" rpy="0 0 1.57" />
   </joint>
 </robot>
